File: breakouts.brd (EAGLE design)
At the start: 160 x 100 mm, 17 parts, among them J1 RJ11, J2 POWERPOLE_POWER25A, X1 NC3FAH2-0

Commit message: minor changes for gerber generation
Other:
- board size 160 x 100 mm -> 46.5 x 47.5 mm
Changed lines of the file:
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@@
 <board>
 <plain>
-<wire x1="0" y1="0" x2="160" y2="0" width="0" layer="20"/>
-<wire x1="160" y1="0" x2="160" y2="100" width="0" layer="20"/>
-<wire x1="160" y1="100" x2="0" y2="100" width="0" layer="20"/>
-<wire x1="0" y1="100" x2="0" y2="0" width="0" layer="20"/>
-<dimension x1="0" y1="0" x2="50" y2="0" x3="25" y3="-9" textsize="1.778" layer="20"/>
-<dimension x1="0" y1="0" x2="0" y2="50" x3="-19" y3="25" textsize="1.778" layer="20"/>
+<dimension x1="0" y1="0" x2="50" y2="0" x3="25" y3="-9" textsize="1.778" layer="49"/>
+<dimension x1="0" y1="0" x2="0" y2="50" x3="-19" y3="25" textsize="1.778" layer="49"/>
 <text x="32.5" y="23.5" size="0.6096" layer="25" font="vector" rot="R90">TUSB320</text>
-<text x="34.5" y="22" size="0.6096" layer="25" font="vector" rot="MR90">INT_N</text>
+<text x="35.5" y="22" size="0.6096" layer="26" font="vector" rot="MR90">INT_N</text>
 <text x="38" y="22" size="0.6096" layer="26" font="vector" rot="MR90">SCL</text>
 <text x="39.5" y="22" size="0.6096" layer="26" font="vector" rot="MR90">SDA</text>
@@
 <param name="rvMicroViaOuter" value="0.25"/>
 <param name="rvMicroViaInner" value="0.25"/>
-<param name="rlMinPadTop" value="0.1mm"/>
+<param name="rlMinPadTop" value="4mil"/>
 <param name="rlMaxPadTop" value="20mil"/>
-<param name="rlMinPadInner" value="10mil"/>
+<param name="rlMinPadInner" value="2mil"/>
 <param name="rlMaxPadInner" value="20mil"/>
-<param name="rlMinPadBottom" value="0.1mm"/>
+<param name="rlMinPadBottom" value="3mil"/>
 <param name="rlMaxPadBottom" value="20mil"/>
 <param name="rlMinViaOuter" value="6mil"/>
@@
 <param name="mvStopFrame" value="1"/>
 <param name="mvCreamFrame" value="0"/>
-<param name="mlMinStopFrame" value="0mil"/>
-<param name="mlMaxStopFrame" value="0mil"/>
+<param name="mlMinStopFrame" value="2mil"/>
+<param name="mlMaxStopFrame" value="2mil"/>
 <param name="mlMinCreamFrame" value="0mil"/>
 <param name="mlMaxCreamFrame" value="0mil"/>
@@
 <via x="39.75" y="21.5" extent="1-16" drill="0.4"/>
 <via x="32.25" y="21.5" extent="1-16" drill="0.4"/>
+<polygon width="0.254" layer="16">
+<vertex x="11.75" y="19.5"/>
+<vertex x="11.75" y="0.75"/>
+<vertex x="29.25" y="0.75"/>
+<vertex x="29.25" y="19.5"/>
+</polygon>
 <wire x1="32.25" y1="21.5" x2="26.95" y2="16.5" width="0" layer="19" extent="1-1"/>
 </signal>
